Commit message: Launch for robot arm

File: catkin_ws/src/ros_experiments_irda/urdf/seven_dof_arm.xacro (robot description, xacro)
@@ -99,5 +99,5 @@
     <link name="base_link">
     <visual>
-        <origin xyz="0 0 0" rpy="1.5708 0 0" /> <!-- rotate PI/2 -->
+        <origin xyz="0 0 0" rpy="${M_PI/2} 0 0" /> <!-- rotate PI/2 -->
         <geometry>
             <box size="0.1 0.1 0.1" />
@@ -106,5 +106,5 @@
     </visual>
     <collision>
-        <origin xyz="0 0 0" rpy="1.5708 0 0" /> <!-- rotate PI/2 -->
+        <origin xyz="0 0 0" rpy="${M_PI/2} 0 0" /> <!-- rotate PI/2 -->
         <geometry>
             <box size="0.1 0.1 0.1" />
@@ -119,5 +119,5 @@
         <parent link="base_link" />
         <child link="shoulder_pan_link" />
-        <origin xyz="0 0 0.05" rpy="0 1.5708 ${M_PI*0}" />
+        <origin xyz="0 0 0.05" rpy="0 ${M_PI/2} ${M_PI*0}" />
         <axis xyz="-1 0 0" />
         <limit effort="300" velocity="1" lower="-2.61799387799" upper="1.98394848567" />
@@ -128,14 +128,14 @@
     <link name="shoulder_pan_link">
     <visual>
-        <origin xyz="0 0 0" rpy="0 1.5708 0" />
-        <geometry>
-            <cylinder radius="0.04" length="0.08" />
+        <origin xyz="0 0 0" rpy="0 ${M_PI/2} 0" />
+        <geometry>
+            <cylinder radius="${shoulder_pan_width}" length="${shoulder_pan_len}" />
         </geometry>
         <material name="Red" />
     </visual>
     <collision>
-        <origin xyz="0 0 0" rpy="0 1.5708 0" />
-        <geometry>
-            <cylinder radius="0.04" length="0.08" />
+        <origin xyz="0 0 0" rpy="0 ${M_PI/2} 0" />
+        <geometry>
+            <cylinder radius="${shoulder_pan_width}" length="${shoulder_pan_len}" />
         </geometry>
     </collision>
@@ -148,5 +148,5 @@
         <parent link="shoulder_pan_link" />
         <child link="shoulder_pitch_link" />
-        <origin xyz="-0.041 0.0021 0.0" rpy="-1.5708 0 1.5708" />
+        <origin xyz="-0.041 0.0021 0.0" rpy="-${M_PI/2} 0 ${M_PI/2}" />
         <axis xyz="1 0 0" />
         <limit effort="300" velocity="1" lower="-1.19962513147" upper="1.89994105047" />
@@ -157,5 +157,5 @@
     <link name="shoulder_pitch_link">
     <visual>
-        <origin xyz="-0.002 0 0.04" rpy="0 1.5708 0" />
+        <origin xyz="-0.002 0 0.04" rpy="0 ${M_PI/2} 0" />
         <geometry>
             <box size="${shoulder_pitch_len} ${shoulder_pitch_width} ${shoulder_pitch_height}" />
@@ -164,5 +164,5 @@
     </visual>
     <collision>
-        <origin xyz="-0.002 0 0.04" rpy="0 1.5708 0" />
+        <origin xyz="-0.002 0 0.04" rpy="0 ${M_PI/2} 0" />
         <geometry>
             <box size="${shoulder_pitch_len} ${shoulder_pitch_width} ${shoulder_pitch_height}" />
@@ -177,5 +177,5 @@
         <parent link="shoulder_pitch_link" />
         <child link="elbow_roll_link" />
-        <origin xyz="-0.002 0 0.1206" rpy="${M_PI} 1.5708 0" />
+        <origin xyz="-0.002 0 0.1206" rpy="${M_PI} ${M_PI/2} 0" />
         <axis xyz="-1 0 0" />
         <limit effort="300" velocity="1" lower="-2.61799387799" upper="0.705631162427" />
@@ -186,5 +186,5 @@
     <link name="elbow_roll_link">
     <visual>
-        <origin xyz="-0.015 0.0 -0.0" rpy="0 1.5708 0" />
+        <origin xyz="-0.015 0.0 -0.0" rpy="0 ${M_PI/2} 0" />
         <geometry>
             <cylinder radius="${elbow_roll_width}" length="${elbow_roll_len}" />
@@ -193,5 +193,5 @@
     </visual>
     <collision>
-        <origin xyz="-0.015 0.0 -0.0" rpy="0 1.5708 0" />
+        <origin xyz="-0.015 0.0 -0.0" rpy="0 ${M_PI/2} 0" />
         <geometry>
             <cylinder radius="${elbow_roll_width}" length="${elbow_roll_len}" />
@@ -206,5 +206,5 @@
         <parent link="elbow_roll_link" />
         <child link="elbow_pitch_link" />
-        <origin xyz="-0.035 0 0.0" rpy="0.055 1.5708 0" />
+        <origin xyz="-0.035 0 0.0" rpy="0.055 ${M_PI/2} 0" />
         <axis xyz="1 0 0" />
         <limit effort="300" velocity="1" lower="-1.5953400194" upper="1.93281579274" />
@@ -215,5 +215,5 @@
     <link name="elbow_pitch_link">
     <visual>
-        <origin xyz="0 0 -0.12" rpy="0 1.5708 0" />
+        <origin xyz="0 0 -0.12" rpy="0 ${M_PI/2} 0" />
         <geometry>
             <box size="${elbow_pitch_len} ${elbow_pitch_width} ${elbow_pitch_height}" />
@@ -222,5 +222,5 @@
     </visual>
     <collision>
-        <origin xyz="0 0 -0.12" rpy="0 1.5708 0" />
+        <origin xyz="0 0 -0.12" rpy="0 ${M_PI/2} 0" />
         <geometry>
             <box size="${elbow_pitch_len} ${elbow_pitch_width} ${elbow_pitch_height}" />
@@ -235,5 +235,5 @@
         <parent link="elbow_pitch_link" />
         <child link="wrist_roll_link" />
-        <origin xyz="0.0 0.0081 -.248" rpy="0 1.5708 ${M_PI}" />
+        <origin xyz="0.0 0.0081 -.248" rpy="0 ${M_PI/2} ${M_PI}" />
         <axis xyz="1 0 0" />
         <limit effort="300" velocity="1" lower="-2.61799387799" upper="2.6128806087" />
@@ -243,5 +243,5 @@
     <link name="wrist_roll_link">
     <visual>
-        <origin xyz="0 0 0" rpy="0 1.5708 0" />
+        <origin xyz="0 0 0" rpy="0 ${M_PI/2} 0" />
         <geometry>
             <cylinder radius="${elbow_roll_width}" length="${elbow_roll_len}" />
@@ -250,5 +250,5 @@
     </visual>
     <collision>
-        <origin xyz="0 0 0" rpy="0 1.5708 0" />
+        <origin xyz="0 0 0" rpy="0 ${M_PI/2} 0" />
         <geometry>
             <cylinder radius="${elbow_roll_width}" length="${elbow_roll_len}" />
@@ -263,5 +263,5 @@
         <parent link="wrist_roll_link" />
         <child link="wrist_pitch_link" />
-        <origin xyz="0.0 0.0 0.0001" rpy="0 1.5708 0" />
+        <origin xyz="0.0 0.0 0.0001" rpy="0 ${M_PI/2} 0" />
         <axis xyz="1 0 0" />
         <limit effort="300" velocity="1" lower="-1.5953400194" upper="1.98394848567" />
@@ -272,5 +272,5 @@
     <link name="wrist_pitch_link">
     <visual>
-        <origin xyz="0 0 0.04" rpy="0 1.5708 0" />
+        <origin xyz="0 0 0.04" rpy="0 ${M_PI/2} 0" />
         <geometry>
             <box size="${wrist_pitch_len} ${wrist_pitch_width} ${wrist_pitch_height}" />
@@ -279,5 +279,5 @@
     </visual>
     <collision>
-        <origin xyz="0 0 0.04 " rpy="0 1.5708 0" />
+        <origin xyz="0 0 0.04 " rpy="0 ${M_PI/2} 0" />
         <geometry>
             <box size="${wrist_pitch_len} ${wrist_pitch_width} ${wrist_pitch_height}" />
@@ -304,5 +304,5 @@
     <link name="gripper_roll_link">
     <visual>
-        <origin xyz="0 0 0" rpy="0 1.5708 0" />
+        <origin xyz="0 0 0" rpy="0 ${M_PI/2} 0" />
         <geometry>
             <cylinder radius="${gripper_roll_width}" length="${gripper_roll_len}" />
@@ -311,5 +311,5 @@
     </visual>
     <collision>
-        <origin xyz="0 0 0" rpy="0 1.5708 0" />
+        <origin xyz="0 0 0" rpy="0 ${M_PI/2} 0" />
         <geometry>
             <cylinder radius="${gripper_roll_width}" length="${gripper_roll_len}" />
