Commit message: Diseno de brazo robotico completado - brazo de 7 GDL

File: catkin_ws/src/ros_experiments_irda/urdf/sensors/xtion_pro_live.urdf.xacro (robot description, xacro)
@@ -1,5 +1,5 @@
 <?xml version="1.0"?>
 <robot xmlns:xacro="http://ros.org/wiki/xacro">
-  <xacro:include filename="$(find mastering_ros_robot_description_pkg)/urdf/sensors/xtion_pro_live.gazebo.xacro"/>
+  <xacro:include filename="$(find ros_experiments_irda)/urdf/sensors/xtion_pro_live.gazebo.xacro"/>
   <xacro:macro name="dummy_inertial">
     <inertial>
@@ -31,5 +31,5 @@
           <box size="0.06 0.1 0.03" />
         	-->
-					<mesh filename="package://mastering_ros_robot_description_pkg/meshes/sensors/xtion_pro_live/xtion_pro_live.stl"/>
+					<mesh filename="package://ros_experiments_irda/meshes/sensors/xtion_pro_live/xtion_pro_live.stl"/>
         </geometry>
         <material name="DarkGrey"/>
@@ -37,5 +37,5 @@
       <collision>
       <geometry>
-          <mesh filename="package://mastering_ros_robot_description_pkg/meshes/sensors/xtion_pro_live/xtion_pro_live.dae"/>
+          <mesh filename="package://ros_experiments_irda/meshes/sensors/xtion_pro_live/xtion_pro_live.dae"/>
       </geometry>
       </collision>

File: catkin_ws/src/ros_experiments_irda/urdf/seven_dof_arm.xacro (robot description, xacro)
@@ -1,413 +1,418 @@
 <?xml version="1.0"?>
 <robot name="seven_dof_arm" xmlns:xacro="http://ros.org/wiki/xacro">
-    <!-- Include materials -->
+  <!-- Include materials -->
     <material name="Black">
-        <color rgba="0.0 0.0 0.0 1.0" />
+        <color rgba="0.0 0.0 0.0 1.0"/>
     </material>
     <material name="Red">
-        <color rgba="0.8 0.0 0.0 1.0" />
+        <color rgba="0.8 0.0 0.0 1.0"/>
     </material>
     <material name="White">
-        <color rgba="1.0 1.0 1.0 1.0" />
+        <color rgba="1.0 1.0 1.0 1.0"/>
     </material>
-    <xacro:property name="deg_to_rad" value="0.01745329251994329577" />
-    <!-- Constants -->
-    <xacro:property name="M_SCALE" value="0.001 0.001 0.001" />
-    <xacro:property name="M_PI" value="3.14159" />
-    <!-- Shoulder pan link properties -->
-    <xacro:property name="shoulder_pan_width" value="0.04" />
-    <xacro:property name="shoulder_pan_len" value="0.08" />
-    <!-- Shoulder pitch link properties -->
-    <xacro:property name="shoulder_pitch_len" value="0.14" />
-    <xacro:property name="shoulder_pitch_width" value="0.04" />
-    <xacro:property name="shoulder_pitch_height" value="0.04" />
-    <!-- Elbow roll link properties -->
-    <xacro:property name="elbow_roll_width" value="0.02" />
-    <xacro:property name="elbow_roll_len" value="0.06" />
-    <!-- Elbow pitch link properties -->
-    <xacro:property name="elbow_pitch_len" value="0.22" />
-    <xacro:property name="elbow_pitch_width" value="0.04" />
-    <xacro:property name="elbow_pitch_height" value="0.04" />
-    <!-- Wrist roll link properties -->
-    <xacro:property name="wrist_roll_width" value="0.02" />
-    <xacro:property name="wrist_roll_len" value="0.04" />
-    <!-- wrist pitch link properties -->
-    <xacro:property name="wrist_pitch_len" value="0.06" />
-    <xacro:property name="wrist_pitch_width" value="0.04" />
-    <xacro:property name="wrist_pitch_height" value="0.04" />
-    <!-- Gripper roll link properties -->
-    <xacro:property name="gripper_roll_width" value="0.04" />
-    <xacro:property name="gripper_roll_len" value="0.02" />
-    <!-- Left gripper -->
-    <xacro:property name="left_gripper_len" value="0.08" />
-    <xacro:property name="left_gripper_width" value="0.01" />
-    <xacro:property name="left_gripper_height" value="0.01" />
-    <!-- Right gripper -->
-    <xacro:property name="right_gripper_len" value="0.08" />
-    <xacro:property name="right_gripper_width" value="0.01" />
-    <xacro:property name="right_gripper_height" value="0.01" />
-    <!-- Right gripper -->
-    <xacro:property name="grasp_frame_len" value="0.02" />
-    <xacro:property name="grasp_frame_width" value="0.02" />
-    <xacro:property name="grasp_frame_height" value="0.02" />
-    <xacro:macro name="inertial_matrix" params="mass">
-        <inertial>
-            <mass value="${mass}" />
-            <inertia ixx="1.0" ixy="0.0" ixz="0.0" iyy="0.5" iyz="0.0" izz="1.0" />
-        </inertial>
-    </xacro:macro>
-    <xacro:macro name="transmission_block" params="joint_name">
-        <transmission name="tran1">
-            <type>transmission_interface/SimpleTransmission</type>
-            <joint name="${joint_name}">
-                <hardwareInterface>hardware_interface/PositionJointInterface</hardwareInterface>
-            </joint>
-            <actuator name="motor1">
-                <hardwareInterface>hardware_interface/PositionJointInterface</hardwareInterface>
-                <mechanicalReduction>1</mechanicalReduction>
-            </actuator>
-        </transmission>
-    </xacro:macro>
-    <!-- BOTTOM FIXED LINK
-This link is the base of the arm in which arm is placed -->
-    <!-- ///////////////////////////////////////////////////////////////////////////////////////////////////////////////////// -->
-    <joint name="bottom_joint" type="fixed">
-        <origin xyz="0 0 0" rpy="0 0 0" />
-        <parent link="base_link" />
-        <child link="bottom_link" />
-    </joint>
-    <link name="bottom_link">
-    <visual>
-        <origin xyz=" 0 0 -0.04" rpy="0 0 0" />
-        <geometry>
-            <box size="1 1 0.02" />
-        </geometry>
-        <material name="Brown" />
-    </visual>
-    <collision>
-        <origin xyz=" 0 0 -0.04" rpy="0 0 0" />
-        <geometry>
-            <box size="1 1 0.02" />
-        </geometry>
-    </collision>
-    </link>
-    <gazebo reference="bottom_link">
-        <material>Gazebo/White</material>
-    </gazebo>
-    <!-- ///////////////////////////////////////////////////////////////////////////////////////////////////////////////////// -->
-    <!-- BASE LINK -->
-    <link name="base_link">
-    <visual>
-        <origin xyz="0 0 0" rpy="${M_PI/2} 0 0" /> <!-- rotate PI/2 -->
-        <geometry>
-            <box size="0.1 0.1 0.1" />
-        </geometry>
-        <material name="White" />
-    </visual>
-    <collision>
-        <origin xyz="0 0 0" rpy="${M_PI/2} 0 0" /> <!-- rotate PI/2 -->
-        <geometry>
-            <box size="0.1 0.1 0.1" />
-        </geometry>
-    </collision>
-    <xacro:inertial_matrix mass="1" />
-    </link>
-    <gazebo reference="base_link">
-        <material>Gazebo/White</material>
-    </gazebo>
-    <joint name="shoulder_pan_joint" type="revolute">
-        <parent link="base_link" />
-        <child link="shoulder_pan_link" />
-        <origin xyz="0 0 0.05" rpy="0 ${M_PI/2} ${M_PI*0}" />
-        <axis xyz="-1 0 0" />
-        <limit effort="300" velocity="1" lower="-2.61799387799" upper="1.98394848567" />
-        <dynamics damping="50" friction="1" />
-    </joint>
-    <!-- ///////////////////////////////////////////////////////////////////////////////////////////////////////////////////// -->
-    <!-- SHOULDER PAN LINK -->
-    <link name="shoulder_pan_link">
-    <visual>
-        <origin xyz="0 0 0" rpy="0 ${M_PI/2} 0" />
-        <geometry>
-            <cylinder radius="${shoulder_pan_width}" length="${shoulder_pan_len}" />
-        </geometry>
-        <material name="Red" />
-    </visual>
-    <collision>
-        <origin xyz="0 0 0" rpy="0 ${M_PI/2} 0" />
-        <geometry>
-            <cylinder radius="${shoulder_pan_width}" length="${shoulder_pan_len}" />
-        </geometry>
-    </collision>
-    <xacro:inertial_matrix mass="1" />
-    </link>
-    <gazebo reference="shoulder_pan_link">
-        <material>Gazebo/Red</material>
-    </gazebo>
-    <joint name="shoulder_pitch_joint" type="revolute">
-        <parent link="shoulder_pan_link" />
-        <child link="shoulder_pitch_link" />
-        <origin xyz="-0.041 0.0021 0.0" rpy="-${M_PI/2} 0 ${M_PI/2}" />
-        <axis xyz="1 0 0" />
-        <limit effort="300" velocity="1" lower="-1.19962513147" upper="1.89994105047" />
-        <dynamics damping="50" friction="1" />
-    </joint>
-    <!-- ///////////////////////////////////////////////////////////////////////////////////////////////////////////////////// -->
-    <!-- SHOULDER PITCH LINK -->
-    <link name="shoulder_pitch_link">
-    <visual>
-        <origin xyz="-0.002 0 0.04" rpy="0 ${M_PI/2} 0" />
-        <geometry>
-            <box size="${shoulder_pitch_len} ${shoulder_pitch_width} ${shoulder_pitch_height}" />
-        </geometry>
-        <material name="White" />
-    </visual>
-    <collision>
-        <origin xyz="-0.002 0 0.04" rpy="0 ${M_PI/2} 0" />
-        <geometry>
-            <box size="${shoulder_pitch_len} ${shoulder_pitch_width} ${shoulder_pitch_height}" />
-        </geometry>
-    </collision>
-    <xacro:inertial_matrix mass="1" />
-    </link>
-    <gazebo reference="shoulder_pitch_link">
-        <material>Gazebo/White</material>
-    </gazebo>
-    <joint name="elbow_roll_joint" type="revolute">
-        <parent link="shoulder_pitch_link" />
-        <child link="elbow_roll_link" />
-        <origin xyz="-0.002 0 0.1206" rpy="${M_PI} ${M_PI/2} 0" />
-        <axis xyz="-1 0 0" />
-        <limit effort="300" velocity="1" lower="-2.61799387799" upper="0.705631162427" />
-        <dynamics damping="50" friction="1" />
-    </joint>
-    <!-- ///////////////////////////////////////////////////////////////////////////////////////////////////////////////////// -->
-    <!-- ELBOW ROLL LINK -->
-    <link name="elbow_roll_link">
-    <visual>
-        <origin xyz="-0.015 0.0 -0.0" rpy="0 ${M_PI/2} 0" />
-        <geometry>
-            <cylinder radius="${elbow_roll_width}" length="${elbow_roll_len}" />
-        </geometry>
-        <material name="Black" />
-    </visual>
-    <collision>
-        <origin xyz="-0.015 0.0 -0.0" rpy="0 ${M_PI/2} 0" />
-        <geometry>
-            <cylinder radius="${elbow_roll_width}" length="${elbow_roll_len}" />
-        </geometry>
-    </collision>
-    <xacro:inertial_matrix mass="1" />
-    </link>
-    <gazebo reference="elbow_roll_link">
-        <material>Gazebo/Black</material>
-    </gazebo>
-    <joint name="elbow_pitch_joint" type="revolute">
-        <parent link="elbow_roll_link" />
-        <child link="elbow_pitch_link" />
-        <origin xyz="-0.035 0 0.0" rpy="0.055 ${M_PI/2} 0" />
-        <axis xyz="1 0 0" />
-        <limit effort="300" velocity="1" lower="-1.5953400194" upper="1.93281579274" />
-        <dynamics damping="50" friction="1" />
-    </joint>
-    <!-- ///////////////////////////////////////////////////////////////////////////////////////////////////////////////////// -->
-    <!-- ELBOW PITCH LINK -->
-    <link name="elbow_pitch_link">
-    <visual>
-        <origin xyz="0 0 -0.12" rpy="0 ${M_PI/2} 0" />
-        <geometry>
-            <box size="${elbow_pitch_len} ${elbow_pitch_width} ${elbow_pitch_height}" />
-        </geometry>
-        <material name="Red" />
-    </visual>
-    <collision>
-        <origin xyz="0 0 -0.12" rpy="0 ${M_PI/2} 0" />
-        <geometry>
-            <box size="${elbow_pitch_len} ${elbow_pitch_width} ${elbow_pitch_height}" />
-        </geometry>
-    </collision>
-    <xacro:inertial_matrix mass="1" />
-    </link>
-    <gazebo reference="elbow_pitch_link">
-        <material>Gazebo/Red</material>
-    </gazebo>
-    <joint name="wrist_roll_joint" type="revolute">
-        <parent link="elbow_pitch_link" />
-        <child link="wrist_roll_link" />
-        <origin xyz="0.0 0.0081 -.248" rpy="0 ${M_PI/2} ${M_PI}" />
-        <axis xyz="1 0 0" />
-        <limit effort="300" velocity="1" lower="-2.61799387799" upper="2.6128806087" />
-        <dynamics damping="50" friction="1" />
-    </joint>
-    <!-- WRIST ROLL LINK -->
-    <link name="wrist_roll_link">
-    <visual>
-        <origin xyz="0 0 0" rpy="0 ${M_PI/2} 0" />
-        <geometry>
-            <cylinder radius="${elbow_roll_width}" length="${elbow_roll_len}" />
-        </geometry>
-        <material name="Black" />
-    </visual>
-    <collision>
-        <origin xyz="0 0 0" rpy="0 ${M_PI/2} 0" />
-        <geometry>
-            <cylinder radius="${elbow_roll_width}" length="${elbow_roll_len}" />
-        </geometry>
-    </collision>
-    <xacro:inertial_matrix mass="1" />
-    </link>
-    <gazebo reference="wrist_roll_link">
-        <material>Gazebo/Black</material>
-    </gazebo>
-    <joint name="wrist_pitch_joint" type="revolute">
-        <parent link="wrist_roll_link" />
-        <child link="wrist_pitch_link" />
-        <origin xyz="0.0 0.0 0.0001" rpy="0 ${M_PI/2} 0" />
-        <axis xyz="1 0 0" />
-        <limit effort="300" velocity="1" lower="-1.5953400194" upper="1.98394848567" />
-        <dynamics damping="50" friction="1" />
-    </joint>
-    <!-- ///////////////////////////////////////////////////////////////////////////////////////////////////////////////////// -->
-    <!-- WRIST PITCH LINK -->
-    <link name="wrist_pitch_link">
-    <visual>
-        <origin xyz="0 0 0.04" rpy="0 ${M_PI/2} 0" />
-        <geometry>
-            <box size="${wrist_pitch_len} ${wrist_pitch_width} ${wrist_pitch_height}" />
-        </geometry>
-        <material name="White" />
-    </visual>
-    <collision>
-        <origin xyz="0 0 0.04 " rpy="0 ${M_PI/2} 0" />
-        <geometry>
-            <box size="${wrist_pitch_len} ${wrist_pitch_width} ${wrist_pitch_height}" />
-        </geometry>
-    </collision>
-    <xacro:inertial_matrix mass="1" />
-    </link>
-    <gazebo reference="wrist_pitch_link">
-        <material>Gazebo/White</material>
-    </gazebo>
-    <joint name="gripper_roll_joint" type="revolute">
-        <parent link="wrist_pitch_link" />
-        <child link="gripper_roll_link" />
-        <origin xyz="0 0 0.080" rpy="${1.5*M_PI} -${.5*M_PI} 0" />
-        <axis xyz="1 0 0" />
-        <!--
+    <material name="Brown">
+        <color rgba="1.0 0.7 0.3 1.0"/>
+    </material>
+  <xacro:property name="deg_to_rad" value="0.01745329251994329577"/>
+  <!-- Constants -->
+  <xacro:property name="M_SCALE" value="0.001 0.001 0.001"/>
+  <xacro:property name="M_PI" value="3.14159"/>
+  <!-- Shoulder pan link properties -->
+  <xacro:property name="shoulder_pan_width" value="0.04" />
+  <xacro:property name="shoulder_pan_len" value="0.08" />
+  <!-- Shoulder pitch link properties -->
+  <xacro:property name="shoulder_pitch_len" value="0.14" />
+  <xacro:property name="shoulder_pitch_width" value="0.04" />
+  <xacro:property name="shoulder_pitch_height" value="0.04" />
+  <!-- Elbow roll link properties -->
+  <xacro:property name="elbow_roll_width" value="0.02" />
+  <xacro:property name="elbow_roll_len" value="0.06" />
+  <!-- Elbow pitch link properties -->
+  <xacro:property name="elbow_pitch_len" value="0.22" />
+  <xacro:property name="elbow_pitch_width" value="0.04" />
+  <xacro:property name="elbow_pitch_height" value="0.04" />
+  <!-- Wrist roll link properties -->
+  <xacro:property name="wrist_roll_width" value="0.02" />
+  <xacro:property name="wrist_roll_len" value="0.04" />
+  <!-- wrist pitch link properties -->
+  <xacro:property name="wrist_pitch_len" value="0.06" />
+  <xacro:property name="wrist_pitch_width" value="0.04" />
+  <xacro:property name="wrist_pitch_height" value="0.04" />
+  <!-- Gripper roll link properties -->
+  <xacro:property name="gripper_roll_width" value="0.04" />
+  <xacro:property name="gripper_roll_len" value="0.02" />
+  <!-- Left gripper -->
+  <xacro:property name="left_gripper_len" value="0.08" />
+  <xacro:property name="left_gripper_width" value="0.01" />
+  <xacro:property name="left_gripper_height" value="0.01" />
+  <!-- Right gripper -->
+  <xacro:property name="right_gripper_len" value="0.08" />
+  <xacro:property name="right_gripper_width" value="0.01" />
+  <xacro:property name="right_gripper_height" value="0.01" />
+  <!-- Right gripper -->
+  <xacro:property name="grasp_frame_len" value="0.02" />
+  <xacro:property name="grasp_frame_width" value="0.02" />
+  <xacro:property name="grasp_frame_height" value="0.02" />
+   <xacro:macro name="inertial_matrix" params="mass">
+      <inertial>
+      	<mass value="${mass}" />
+        <inertia ixx="1.0" ixy="0.0" ixz="0.0" iyy="0.5" iyz="0.0" izz="1.0" />
+      </inertial>
+   </xacro:macro>
+   <xacro:macro name="transmission_block" params="joint_name">
+	  <transmission name="tran1">
+	    <type>transmission_interface/SimpleTransmission</type>
+	    <joint name="${joint_name}">
+	      <hardwareInterface>hardware_interface/PositionJointInterface</hardwareInterface>
+	    </joint>
+	    <actuator name="motor1">
+	      <hardwareInterface>hardware_interface/PositionJointInterface</hardwareInterface>
+	      <mechanicalReduction>1</mechanicalReduction>
+	    </actuator>
+	  </transmission>
+   </xacro:macro>
+<!-- BOTTOM FIXED LINK
+This link is the base of the arm in which arm is placed
+-->
+<!-- ///////////////////////////////////////////////////////////////////////////////////////////////////////////////////// -->
+  <joint name="bottom_joint" type="fixed">
+    <origin xyz="0 0 0" rpy="0 0 0" />
+    <parent link="base_link"/>
+    <child link="bottom_link"/>
+  </joint>
+  <link name="bottom_link">
+    <visual>
+      <origin xyz=" 0 0 -0.04"  rpy="0 0 0"/>
+      <geometry>
+	       <box size="1 1 0.02" />
+      </geometry>
+      <material name="Brown" />
+    </visual>
+    <collision>
+      <origin xyz=" 0 0 -0.04"  rpy="0 0 0"/>
+      <geometry>
+	       <box size="1 1 0.02" />
+      </geometry>
+      </collision>
+  </link>
+  <gazebo reference="bottom_link">
+    <material>Gazebo/White</material>
+  </gazebo>
+<!-- ///////////////////////////////////////////////////////////////////////////////////////////////////////////////////// -->
+  <!-- BASE LINK -->
+  <link name="base_link">
+    <visual>
+      <origin xyz="0 0 0" rpy="${M_PI/2} 0 0" /> <!-- rotate PI/2 -->
+      <geometry>
+	       <box size="0.1 0.1 0.1" />
+      </geometry>
+      <material name="White" />
+    </visual>
+    <collision>
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